File: KiCad/project/project.kicad_pcb (KiCad board)
At the start: 4 copper layers, 40 x 45 mm, 29 parts, among them P1 TB002-500-05BE, U1 DRV8313PWPR

Commit message: PCB: re-place C3/C5 to the Ø10mm footprint (50x45 board); fixes part/footprint mismatch
C3/C5's BOM part C87862 (RVT2A470M1010, 47uF/100V) is a Ø10mm can but the
board had the Ø6.3mm footprint (surfaced by easyeda2kicad). Swapped to
CAP-SMD_BD10.0 and re-laid-out, headless. Electrically clean: 0 error-severity
DRC, 0 unconnected, all nets connected; schematic C3/C5 footprint synced.

- Enlarged 40x45 -> 50x45 (within the <=50x50 budget); relocated P1 + MH2/MH3
  to the new right edge (rest of the board untouched).
- Added CAP-SMD_BD10.0 to simplefocmini.pretty (from the easyeda2kicad download);
  swapped C3/C5 footprints (pad nets re-bound by name).
- Placed both cans rot90, stacked on the right, spread to clear the divider and
  the P1 fan; routed the phase/VM nets under the SMD cans on B.Cu. Autorouter was
  unstable on this congested area -> deterministic hand-route for the last mile.
- Re-poured In1/In2 GND planes to the new outline (inset to clear rounded corners).

Note: kicad-cli pcb drc normalises project.kicad_pro and resets the custom
min-via rules (0.4/0.25/0.075) -> false via violations; restored values, verified
clean with KiCadRoutingTools check_drc.py + check_connected.

Co-Authored-By: Claude Opus 4.8 (1M context) <noreply@anthropic.com>
Parts:
- C3, C5: footprint simplefocmini:CAP-SMD_BD6.3-L6.6-W6.6-FD -> simplefocmini:CAP-SMD_BD10.0-L10.3-W10.3-FD-LS11.0
- moved C3 27.8 mm to (168.6, 97.5), turned to 90 degrees
- moved C5 23.7 mm to (168.6, 119.0), turned to 90 degrees
- moved MH2 10.0 mm to (180.0, 92.0)
- moved MH3 10.0 mm to (180.0, 129.0)
- moved P1 10.0 mm to (179.0, 120.5)
Routing:
- net M3: track 17.8 -> 27.8 mm, vias 2 -> 4
- net M2: track 16.4 -> 25.6 mm, vias 0 -> 1
- net M1: track 18.2 -> 26.9 mm, vias 0 -> 1
- net VCC: track 84.2 -> 83.5 mm
- net GND: vias 11 -> 13
Other:
- board size 40 x 45 mm -> 50 x 45 mm

Commit message: Silk: rebrand SimpleFOC Mini -> DRV8313
Renamed the PCB silkscreen branding (top + bottom) from 'SimpleFOC Mini v2.0' to 'DRV8313', updated the doc URL to the new repo and the date; regenerated the silk gerbers, PCB SVGs, and 3D renders to match. 0 error-severity DRC, unchanged otherwise.

Co-Authored-By: Claude Opus 4.8 (1M context) <noreply@anthropic.com>
Other:
- board text added: "06/26"
- board text added: "Board v2.0"
- board text added: "DRV8313"
- board text added: "github.com/kaydensigh/drv8313-board"
- board text removed: "04/24"
- board text removed: "Mini"
- board text removed: "Mini v2.0"
- board text removed: "SimpleFOC"
- board text removed: "docs.simplefoc.com"
Changed lines of the file:
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@@
 		)
 	)
-	(gr_text "Mini"
-		(at 155.3 117 0)
+	(gr_text "DRV8313"
+		(at 157 115.3 0)
 		(layer "F.SilkS")
 		(effects
@@
 		)
 	)
-	(gr_text "SimpleFOC"
-		(at 157 115.3 0)
+	(gr_text "v2.0"
+		(at 157 117 0)
 		(layer "F.SilkS")
 		(effects
@@
 	(gr_text "8-60V"
 		(at 157 118.7 0)
-		(layer "F.SilkS")
-		(effects
-			(font
-				(size 0.8 0.8)
-				(thickness 0.13)
-			)
-			(justify top)
-		)
-	)
-	(gr_text "v2.0"
-		(at 158.6 117 0)
 		(layer "F.SilkS")
 		(effects
@@
 		)
 	)
-	(gr_text "docs.simplefoc.com"
+	(gr_text "github.com/kaydensigh/drv8313-board"
 		(at 149 131 0)
 		(layer "B.SilkS")
@@
 		)
 	)
-	(gr_text "SimpleFOC"
+	(gr_text "DRV8313"
 		(at 140 118.5 0)
 		(layer "B.SilkS")
@@
 		)
 	)
-	(gr_text "Mini v2.0"
+	(gr_text "Board v2.0"
 		(at 140 120.3 0)
 		(layer "B.SilkS")
@@
 		)
 	)
-	(gr_text "04/24"
+	(gr_text "06/26"
 		(at 140 122.1 0)
 		(layer "B.SilkS")

Commit message: Silk: version v2.0 -> v1.0 (first release as drv8313-board)
Co-Authored-By: Claude Opus 4.8 (1M context) <noreply@anthropic.com>
Other:
- board text added: "Board v1.0"
- board text added: "v1.0"
- board text removed: "Board v2.0"
- board text removed: "v2.0"
Changed lines of the file:
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@@
 		)
 	)
-	(gr_text "v2.0"
+	(gr_text "v1.0"
 		(at 157 117 0)
 		(layer "F.SilkS")
@@
 		)
 	)
-	(gr_text "Board v2.0"
+	(gr_text "Board v1.0"
 		(at 140 120.3 0)
 		(layer "B.SilkS")

Commit message: BOM: source all parts (JLCPCB Basic-preferred) + 3D models so all parts render
BOM (manufacturing/drv8313-board-BOM.csv) - fill every blank MPN/LCSC and fix
two import-era errors:
- R1-R4 carried the 4.7k part C23162 despite a 10k value -> C25804 (Basic)
- P1's C146243 was actually a 3-pin header, not the 5-pos block -> DB126V-5.0-5P (C2835160)
Filled: R6/R7/R12 10k C25804, R9 43k C23172, R10 62k C23221, R11 1k C21190,
R8 50mOhm 3W shunt C2903475, C6 470nF C1623 (= C4), H1 2x7 socket C38844,
TB_PWR1 2-pos block C395849. Values normalized so identical parts group;
PCB value text synced to match.

3D render - the project-local footprints referenced 3D models in directories
that were never committed (EASYEDA_MODELS / a deleted scratch dir), so U1, the
0603 passives, the LED and both cans dropped out of the render. Fetched the
exact models with easyeda2kicad into KiCad/project/EASYEDA_MODELS/ and repointed
every (model) to the committed .wrl. Terminal blocks (KiCad ships no 3D for the
MaiXu series here) got Degson DB126V models attached to the footprints.

Regenerated images/board-3d-{top,bottom}.png, images/schematic.svg and
manufacturing/drv8313-board.step (--subst-models). DRC 0 violations, all 27
nets connected, ERC at the 141 baseline. Docs updated (README, redesign-bom,
CLAUDE).

Co-Authored-By: Claude Opus 4.8 (1M context) <noreply@anthropic.com>
Parts:
- C6: value 0.47uF -> 470nF
- P1: value TB002-500-05BE -> TerminalBlock 5P 5.0mm
- R10: value 62k -> 62kΩ
- R11: value 1k -> 1kΩ
- R12, R6, R7: value 10k -> 10kΩ
- R8: value 0.05 -> 50mΩ
- R9: value 43k -> 43kΩ
- TB_PWR1: value TB002-500-02BE -> TerminalBlock 2P 5.0mm
Changed lines of the file:
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@@
 			)
 		)
-		(property "Value" "0.47uF"
+		(property "Value" "470nF"
 			(at 4.0792 -3.0963 270)
 			(layer "F.SilkS")
@@
 		)
 		(embedded_fonts no)
-		(model "${KIPRJMOD}/EASYEDA_MODELS/C0603_L1.6-W0.8-H0.8.step"
+		(model "${KIPRJMOD}/EASYEDA_MODELS/C0603_L1.6-W0.8-H0.8.wrl"
 			(offset
 				(xyz 0 0 0)
@@
 		)
 		(embedded_fonts no)
-		(model "${KIPRJMOD}/EASYEDA_MODELS/R0603_L1.6-W0.8-H0.8.step"
+		(model "${KIPRJMOD}/EASYEDA_MODELS/R0603.wrl"
 			(offset
 				(xyz 0 -0 0)
@@
 		)
 		(embedded_fonts no)
-		(model "${KIPRJMOD}/EASYEDA_MODELS/C0603_L1.6-W0.8-H0.8.step"
+		(model "${KIPRJMOD}/EASYEDA_MODELS/C0603_L1.6-W0.8-H0.8.wrl"
 			(offset
 				(xyz 0 0 0)
@@
 			)
 		)
-		(property "Value" "10k"
+		(property "Value" "10kΩ"
 			(at 2.4511 -4.3383 180)
 			(layer "F.SilkS")
@@
 		)
 		(embedded_fonts no)
-		(model "${KIPRJMOD}/EASYEDA_MODELS/R0603_L1.6-W0.8-H0.8.step"
+		(model "${KIPRJMOD}/EASYEDA_MODELS/R0603.wrl"
 			(offset
 				(xyz 0 0 0)
@@
 			)
 		)
-		(property "Value" "TB002-500-02BE"
+		(property "Value" "TerminalBlock 2P 5.0mm"
 			(at 2.25 4.92 90)
 			(layer "F.Fab")
@@
 		)
 		(embedded_fonts no)
-		(model "${KICAD10_3DMODEL_DIR}/TerminalBlock.3dshapes/TerminalBlock_MaiXu_MX126-5.0-02P_1x02_P5.00mm.step"
+		(model "${KIPRJMOD}/EASYEDA_MODELS/CONN-TH_DB5.00-LI-2P-126.wrl"
 			(offset
-				(xyz 0 0 0)
+				(xyz 2.5 0 0)
 			)
 			(scale
@@
 			)
 			(rotate
-				(xyz 0 0 0)
+				(xyz 0 0 180)
 			)
 		)
@@
 			)
 		)
-		(property "Value" "43k"
+		(property "Value" "43kΩ"
 			(at 2.4511 -4.3383 270)
 			(layer "F.SilkS")
@@
 		)
 		(embedded_fonts no)
-		(model "${KIPRJMOD}/EASYEDA_MODELS/R0603_L1.6-W0.8-H0.8.step"
+		(model "${KIPRJMOD}/EASYEDA_MODELS/R0603.wrl"
 			(offset
 				(xyz 0 0 0)
@@
 			)
 		)
-		(property "Value" "TB002-500-05BE"
+		(property "Value" "TerminalBlock 5P 5.0mm"
 			(at 9.75 4.92 90)
 			(layer "F.Fab")
@@
 		)
 		(embedded_fonts no)
-		(model "${KICAD10_3DMODEL_DIR}/TerminalBlock.3dshapes/TerminalBlock_MaiXu_MX126-5.0-05P_1x05_P5.00mm.step"
+		(model "${KIPRJMOD}/EASYEDA_MODELS/CONN-TH_5P-P5.00-L8.0-W25.0.wrl"
 			(offset
-				(xyz 0 0 0)
+				(xyz 10.0 0 0)
 			)
 			(scale
@@
 			)
 			(rotate
-				(xyz 0 0 0)
+				(xyz 0 0 180)
 			)
 		)
@@
 		)
 		(embedded_fonts no)
-		(model "${KIPRJMOD}/EASYEDA_MODELS/HTSSOP-28_L9.7-W4.4-H1.2-LS6.4-P0.65.step"
+		(model "${KIPRJMOD}/EASYEDA_MODELS/HTSSOP-28_L9.7-W4.4-H1.2-LS6.4-P0.65.wrl"
 			(offset
 				(xyz -0 0.0001 0)
@@
 		)
 		(embedded_fonts no)
-		(model "${KIPRJMOD}/EASYEDA_MODELS/C0603_L1.6-W0.8-H0.8.step"
+		(model "${KIPRJMOD}/EASYEDA_MODELS/C0603_L1.6-W0.8-H0.8.wrl"
 			(offset
 				(xyz 0 -0 0)
@@
 		)
 		(embedded_fonts no)
-		(model "${KIPRJMOD}/EASYEDA_MODELS/R0603_L1.6-W0.8-H0.8.step"
+		(model "${KIPRJMOD}/EASYEDA_MODELS/R0603.wrl"
 			(offset
 				(xyz 0 0 0)
@@
 			)
 		)
-		(property "Value" "10k"
+		(property "Value" "10kΩ"
 			(at 2.4511 -4.3383 270)
 			(layer "F.SilkS")
@@
 		)
 		(embedded_fonts no)
-		(model "${KIPRJMOD}/EASYEDA_MODELS/R0603_L1.6-W0.8-H0.8.step"
+		(model "${KIPRJMOD}/EASYEDA_MODELS/R0603.wrl"
 			(offset
 				(xyz 0 0 0)
@@
 			)
 		)
-		(property "Value" "0.05"
+		(property "Value" "50mΩ"
 			(at 0 2.63 180)
 			(layer "F.Fab")
@@
 			)
 		)
-		(property "Value" "10k"
+		(property "Value" "10kΩ"
 			(at 2.4511 -4.3383 0)
 			(layer "F.SilkS")
@@
 		)
 		(embedded_fonts no)
-		(model "${KIPRJMOD}/EASYEDA_MODELS/R0603_L1.6-W0.8-H0.8.step"
+		(model "${KIPRJMOD}/EASYEDA_MODELS/R0603.wrl"
 			(offset
 				(xyz 0 0 0)
@@
 		)
 		(embedded_fonts no)
-		(model "${KIPRJMOD}/EASYEDA_MODELS/R0603_L1.6-W0.8-H0.8.step"
+		(model "${KIPRJMOD}/EASYEDA_MODELS/R0603.wrl"
 			(offset
 				(xyz 0 0 0)
@@
 		)
 		(embedded_fonts no)
-		(model "_scratch_ee/sfm.3dshapes/CAP-SMD_BD10.0-L10.3-W10.3-FD-LS11.0.wrl"
+		(model "${KIPRJMOD}/EASYEDA_MODELS/CAP-SMD_BD10.0-L10.3-W10.3-FD-LS11.0.wrl"
 			(offset
 				(xyz 0 0 0)
@@
 		)
 		(embedded_fonts no)
-		(model "${KIPRJMOD}/EASYEDA_MODELS/R0603_L1.6-W0.8-H0.8.step"
+		(model "${KIPRJMOD}/EASYEDA_MODELS/R0603.wrl"
 			(offset
 				(xyz 0 0 0)
@@
 			)
 		)
-		(property "Value" "62k"
+		(property "Value" "62kΩ"
 			(at 2.4511 -4.3383 180)
 			(layer "F.SilkS")
@@
 		)
 		(embedded_fonts no)
-		(model "${KIPRJMOD}/EASYEDA_MODELS/R0603_L1.6-W0.8-H0.8.step"
+		(model "${KIPRJMOD}/EASYEDA_MODELS/R0603.wrl"
 			(offset
 				(xyz 0 0 0)
@@
 			)
 		)
-		(property "Value" "1k"
+		(property "Value" "1kΩ"
 			(at 2.4511 -4.3383 0)
 			(layer "F.SilkS")
@@
 		)
 		(embedded_fonts no)
-		(model "${KIPRJMOD}/EASYEDA_MODELS/R0603_L1.6-W0.8-H0.8.step"
+		(model "${KIPRJMOD}/EASYEDA_MODELS/R0603.wrl"
 			(offset
 				(xyz 0 0 0)
@@
 		)
 		(embedded_fonts no)
-		(model "${KIPRJMOD}/EASYEDA_MODELS/R0603_L1.6-W0.8-H0.8.step"
+		(model "${KIPRJMOD}/EASYEDA_MODELS/R0603.wrl"
 			(offset
 				(xyz -0 0 0)
@@
 		)
 		(embedded_fonts no)
-		(model "${KIPRJMOD}/EASYEDA_MODELS/LED0603_L1.6-W0.8-H0.6.step"
+		(model "${KIPRJMOD}/EASYEDA_MODELS/LED0603-RD-YELLOW.wrl"
 			(offset
 				(xyz -0 0 0)
@@
 		)
 		(embedded_fonts no)
-		(model "${KIPRJMOD}/EASYEDA_MODELS/C0603_L1.6-W0.8-H0.8.step"
+		(model "${KIPRJMOD}/EASYEDA_MODELS/C0603_L1.6-W0.8-H0.8.wrl"
 			(offset
 				(xyz 0 0 0)
@@
 		)
 		(embedded_fonts no)
-		(model "_scratch_ee/sfm.3dshapes/CAP-SMD_BD10.0-L10.3-W10.3-FD-LS11.0.wrl"
+		(model "${KIPRJMOD}/EASYEDA_MODELS/CAP-SMD_BD10.0-L10.3-W10.3-FD-LS11.0.wrl"
 			(offset
 				(xyz 0 0 0)

Commit message: Tools: add JLCPCB part search + fab/silk scripts; re-source 2 BOM parts
Add tools/ headless helpers (see tools/README.md):
- jlc_search.py: live JLCPCB part finder. Ranks fee-free first (Basic OR
  Preferred -- both incur no per-part setup fee) then cheapest in-stock.
  Uses the API's server-side library filters (--fee-free/--basic/--preferred),
  which surface no-fee parts that plain keyword search buries behind Extended.
- build_manufacturing.py: regenerate gerbers/drill/zip/CPL/BOM/STEP + images
  in one command; snapshots/restores project.kicad_pro (kicad-cli rewrites it).
- set_silk_version.py: bump the vN.M (+ MM/YY) silkscreen stamp.

BOM cost/availability pass (jlc_search.py), non-geometric:
- C2 100nF C1591 (Extended) -> C14663 (YAGEO, Basic): drops a per-part fee;
  like-for-like 50V (netlist confirms C2 spans VCP-VM ~11V).
- LED1 C72038 (yellow, out of stock) -> C89811 (NationStar, yellow, Preferred,
  in stock) -- keeps original colour.
- Confirmed 43k/62k dividers are Preferred (fee-free), not Extended as earlier
  docs claimed; corrected README / redesign-bom / CLAUDE.md.
- Kept the unavoidable Extended parts (U1, 10nF/100V & 47uF/100V caps, 50mR
  shunt, connectors). 10k C25804 is Basic but read stock 0 -- flagged.

0 error-severity DRC, 27/27 nets connected, ERC 141 baseline (unchanged).

Co-Authored-By: Claude Opus 4.8 (1M context) <noreply@anthropic.com>
Parts:
- LED1: value 19-213/Y2C-CQ2R2L/3T(CY) -> Yellow
Changed lines of the file:
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@@
 		(model "${KIPRJMOD}/EASYEDA_MODELS/CONN-TH_5P-P5.00-L8.0-W25.0.wrl"
 			(offset
-				(xyz 10.0 0 0)
+				(xyz 10 0 0)
 			)
 			(scale
@@
 			)
 		)
-		(property "Value" "19-213/Y2C-CQ2R2L/3T(CY)"
+		(property "Value" "Yellow"
 			(at 24.6075 -3.1674 0)
 			(layer "F.SilkS")
