File: KiCad/project/project.kicad_pcb (KiCad board)
At the start: 4 copper layers, 50 x 45 mm, 29 parts, among them P1 TerminalBlock 5P 5.0mm, U1 DRV8313PWPR

Commit message: Claude's attempt at redoing the whole layout.
Parts:
- added C7: 100nF 100V, simplefocmini:C0603, F.Cu at (155.5, 114.0)
- added C8: 100nF 100V, simplefocmini:C0603, F.Cu at (160.5, 114.0)
- moved C3 34.6 mm to (149.0, 126.0)
- moved C4 20.2 mm to (164.5, 106.0)
- moved R2 8.30 mm to (162.3, 100.0)
- moved R4 7.96 mm to (153.8, 100.0)
- moved C6 7.96 mm to (161.4, 123.0)
- moved R6 7.50 mm to (155.5, 100.0)
- moved R10 7.30 mm to (157.8, 123.0)
- moved R7 7.20 mm to (157.2, 100.0)
- moved R5 7.16 mm to (166.5, 103.0)
- moved R8 7.07 mm to (159.0, 118.0)
- moved R12 6.90 mm to (158.9, 100.0)
- moved SJ1 6.51 mm to (155.5, 130.5)
- moved H1 6.15 mm to (151.4, 93.0)
- moved LED1 6.02 mm to (168.0, 100.5)
- moved R11 6.00 mm to (159.6, 123.0)
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Routing:
- net PGND: track 48.6 -> 33.8 mm, vias 7 -> 4
- net IN1: track 26.8 -> 12.1 mm
- net 3.3V: track 77.3 -> 89.6 mm, vias 11 -> 10
- net VCC: track 85.4 -> 97.2 mm, vias 4 -> 3
- net Net-(U1-CP2): track 14.8 -> 5.58 mm, vias 2 -> 0
- net XN: track 3.10 -> 12.3 mm
- net YN: track 4.20 -> 13.0 mm
- net Net-(U1-CP1): track 11.0 -> 3.94 mm, vias 2 -> 0
- net EN1: track 12.7 -> 5.61 mm
- net EN2: track 12.4 -> 5.36 mm
- net nCOMPO: track 17.9 -> 12.0 mm, vias 3 -> 1
- net EN3: track 11.0 -> 5.55 mm, vias 2 -> 0
- net Net-(U1-VCP): track 2.71 -> 8.18 mm, vias 2 -> 0
- net nFlt: track 20.0 -> 14.7 mm, vias 2 -> 4
- net IN2: track 17.8 -> 12.6 mm
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Other:
- board size 50 x 45 mm -> 50 x 50 mm

Commit message: Manual layout.
Parts:
- moved SJ1 31.8 mm to (166.5, 100.7), turned to 0 degrees
- moved SJ2 31.2 mm to (171.0, 100.7), turned to 0 degrees
- moved R11 21.9 mm to (171.0, 104.3)
- moved R10 20.7 mm to (166.5, 104.3), turned to 90 degrees
- moved R9 18.0 mm to (164.7, 107.3), turned to 0 degrees
- moved C6 13.4 mm to (164.8, 110.0), turned to 180 degrees
- moved LED1 9.01 mm to (165.0, 92.0), turned to 0 degrees
- moved R5 8.63 mm to (165.0, 94.5), turned to 0 degrees
- moved C7 8.32 mm to (151.5, 106.7)
- moved R4 7.41 mm to (146.5, 98.7), turned to -90 degrees
- moved R6 6.62 mm to (149.0, 98.8), turned to -90 degrees
- moved H1 6.24 mm to (145.3, 91.5)
- moved R7 5.35 mm to (152.0, 98.8), turned to -90 degrees
- moved C2 4.18 mm to (154.8, 112.5), turned to 180 degrees
- moved R12 4.05 mm to (155.0, 98.8), turned to -90 degrees
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Connections:
- C7 pad 1: VCC -> GND
- C7 pad 2: GND -> VCC
- C8 pad 1: VCC -> GND
- C8 pad 2: GND -> VCC
- H1 pad 1: GND -> IN1
- H1 pad 11: nFlt -> VREF
- H1 pad 12: nCOMPO -> PGND
- H1 pad 13: PGND -> GND
- H1 pad 14: VREF -> 3.3V
- H1 pad 2: 3.3V -> EN1H
- H1 pad 3: IN1 -> IN2
- H1 pad 4: EN1H -> EN2H
- H1 pad 5: IN2 -> IN3
- H1 pad 6: EN2H -> EN3H
- H1 pad 7: IN3 -> nFlt
- H1 pad 8: EN3H -> nCOMPO
- P1 pad 1: GND -> VCC
- P1 pad 5: VCC -> GND
Routing:
- net 3.3V: track 89.6 -> 29.6 mm, vias 10 -> 5
- net VREF: track 64.7 -> 35.0 mm, vias 15 -> 0
- net VCC: track 97.2 -> 79.7 mm, vias 3 -> 0
- net YN: track 13.0 -> 3.12 mm
- net XN: track 12.3 -> 3.12 mm
- net IN1: track 12.1 -> 20.6 mm
- net PGND: track 33.8 -> 42.1 mm, vias 4 -> 1
- net IN2: track 12.6 -> 19.7 mm, vias 2 -> 0
- net EN1: track 5.61 -> 11.3 mm, vias 2 -> 0
- net IN3: track 13.1 -> 18.2 mm, vias 2 -> 0
- net Net-(U1-VCP): track 8.18 -> 3.82 mm
- net EN2: track 5.36 -> 9.70 mm
- net nSlp: track 15.5 -> 12.9 mm, vias 1 -> 0
- net EN3: track 5.55 -> 8.04 mm
- net nRes: track 14.3 -> 16.8 mm, vias 2 -> 0
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