File: KiCad/project/project.kicad_sch (KiCad schematic)
At the start: 27 parts, among them P1 TerminalBlock 5P 5.0mm, U1 DRV8313PWPR

Commit message: Rename project library simplefocmini -> drv8313-board
The board long ago diverged from SimpleFOCMini, so renamed the project KiCad
library nickname (used for both the footprint .pretty and the symbol .kicad_sym)
to match the repo/manufacturing naming.

- Renamed KiCad/project/simplefocmini.pretty -> drv8313-board.pretty and
  simplefocmini.kicad_sym -> drv8313-board.kicad_sym (git mv).
- Updated the project fp-lib-table + sym-lib-table (name + URI), all PCB FPIDs
  (21) and schematic lib_ids/Footprint fields (25), and the BOM Footprint column.
- Updated the lib-name references in README/CLAUDE.md; preserved the legitimate
  SimpleFOCMini attribution, the EasyEDA source URL, and the historical Altium
  filename.

Footprints + symbols re-verified to resolve under the new nickname (parity found
the lib; ERC 0). check_design.py PASS (DRC 0 errors, ERC 0). Netlist/PCB
geometry unchanged; project.kicad_pro untouched.

Co-Authored-By: Claude Opus 4.8 (1M context) <noreply@anthropic.com>
Parts:
- C1, C2, C4, C6, C7, C8: footprint simplefocmini:C0603 -> drv8313-board:C0603
- C3, C5: footprint simplefocmini:CAP-SMD_BD10.0-L10.3-W10.3-FD-LS11.0 -> drv8313-board:CAP-SMD_BD10.0-L10.3-W10.3-FD-LS11.0
- LED1: footprint simplefocmini:LED0603-R-RD -> drv8313-board:LED0603-R-RD; symbol simplefocmini:19-213/Y2C-CQ2R2L/3T(CY) -> drv8313-board:19-213/Y2C-CQ2R2L/3T(CY)
- R1, R10, R11, R12, R2, R3, R4, R5, R6, R7, R9: footprint simplefocmini:R0603 -> drv8313-board:R0603
- U1: footprint simplefocmini:HTSSOP-28_L9.8-W4.5-P0.65-LS6.6-BL-EP -> drv8313-board:HTSSOP-28_L9.8-W4.5-P0.65-LS6.6-BL-EP; symbol simplefocmini:DRV8313PWPR -> drv8313-board:DRV8313PWPR
Changed lines of the file:
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@@
 			)
 		)
-		(property "Footprint" "simplefocmini:R0603"
+		(property "Footprint" "drv8313-board:R0603"
 			(at 205.74 93.98 0)
 			(hide yes)
@@
 			)
 		)
-		(property "Footprint" "simplefocmini:R0603"
+		(property "Footprint" "drv8313-board:R0603"
 			(at 152.4 111.76 0)
 			(hide yes)
@@
 			)
 		)
-		(property "Footprint" "simplefocmini:C0603"
+		(property "Footprint" "drv8313-board:C0603"
 			(at 69.85 71.12 0)
 			(hide yes)
@@
 	)
 	(symbol
-		(lib_id "simplefocmini:DRV8313PWPR")
+		(lib_id "drv8313-board:DRV8313PWPR")
 		(at 152.4 73.66 0)
 		(unit 0)
@@
 			)
 		)
-		(property "Footprint" "simplefocmini:HTSSOP-28_L9.8-W4.5-P0.65-LS6.6-BL-EP"
+		(property "Footprint" "drv8313-board:HTSSOP-28_L9.8-W4.5-P0.65-LS6.6-BL-EP"
 			(at 152.4 73.66 0)
 			(hide yes)
@@
 			)
 		)
-		(property "Footprint" "simplefocmini:R0603"
+		(property "Footprint" "drv8313-board:R0603"
 			(at 208.28 57.15 0)
 			(hide yes)
@@
 			)
 		)
-		(property "Footprint" "simplefocmini:R0603"
+		(property "Footprint" "drv8313-board:R0603"
 			(at 143.51 33.02 0)
 			(hide yes)
@@
 			)
 		)
-		(property "Footprint" "simplefocmini:C0603"
+		(property "Footprint" "drv8313-board:C0603"
 			(at 162.56 119.38 0)
 			(hide yes)
@@
 			)
 		)
-		(property "Footprint" "simplefocmini:C0603"
+		(property "Footprint" "drv8313-board:C0603"
 			(at 127 58.42 0)
 			(hide yes)
@@
 			)
 		)
-		(property "Footprint" "simplefocmini:R0603"
+		(property "Footprint" "drv8313-board:R0603"
 			(at 109.22 106.68 0)
 			(hide yes)
@@
 			)
 		)
-		(property "Footprint" "simplefocmini:C0603"
+		(property "Footprint" "drv8313-board:C0603"
 			(at 116.84 63.5 0)
 			(hide yes)
@@
 	)
 	(symbol
-		(lib_id "simplefocmini:19-213/Y2C-CQ2R2L/3T(CY)")
+		(lib_id "drv8313-board:19-213/Y2C-CQ2R2L/3T(CY)")
 		(at 153.67 121.92 270)
 		(unit 0)
@@
 			)
 		)
-		(property "Footprint" "simplefocmini:LED0603-R-RD"
+		(property "Footprint" "drv8313-board:LED0603-R-RD"
 			(at 153.67 121.92 0)
 			(hide yes)
@@
 			)
 		)
-		(property "Footprint" "simplefocmini:R0603"
+		(property "Footprint" "drv8313-board:R0603"
 			(at 227.33 130.81 0)
 			(hide yes)
@@
 			)
 		)
-		(property "Footprint" "simplefocmini:CAP-SMD_BD10.0-L10.3-W10.3-FD-LS11.0"
+		(property "Footprint" "drv8313-board:CAP-SMD_BD10.0-L10.3-W10.3-FD-LS11.0"
 			(at 71.12 71.12 0)
 			(hide yes)
@@
 			)
 		)
-		(property "Footprint" "simplefocmini:R0603"
+		(property "Footprint" "drv8313-board:R0603"
 			(at 123.19 40.64 0)
 			(hide yes)
@@
 			)
 		)
-		(property "Footprint" "simplefocmini:R0603"
+		(property "Footprint" "drv8313-board:R0603"
 			(at 74.93 120.65 0)
 			(hide yes)
@@
 			)
 		)
-		(property "Footprint" "simplefocmini:CAP-SMD_BD10.0-L10.3-W10.3-FD-LS11.0"
+		(property "Footprint" "drv8313-board:CAP-SMD_BD10.0-L10.3-W10.3-FD-LS11.0"
 			(at 77.47 71.12 0)
 			(hide yes)
@@
 			)
 		)
-		(property "Footprint" "simplefocmini:C0603"
+		(property "Footprint" "drv8313-board:C0603"
 			(at 129.54 148.59 0)
 			(hide yes)
@@
 			)
 		)
-		(property "Footprint" "simplefocmini:C0603"
+		(property "Footprint" "drv8313-board:C0603"
 			(at 63.5 71.12 0)
 			(hide yes)
@@
 			)
 		)
-		(property "Footprint" "simplefocmini:R0603"
+		(property "Footprint" "drv8313-board:R0603"
 			(at 189.23 93.98 0)
 			(hide yes)
@@
 			)
 		)
-		(property "Footprint" "simplefocmini:R0603"
+		(property "Footprint" "drv8313-board:R0603"
 			(at 175.26 93.98 0)
 			(hide yes)
@@
 			)
 		)
-		(property "Footprint" "simplefocmini:R0603"
+		(property "Footprint" "drv8313-board:R0603"
 			(at 104.14 139.7 0)
 			(hide yes)
